File: Hardware/SparkFun_NEO-F10N.kicad_sch (KiCad schematic)
At the start: 49 parts, among them J1 USB_C_Receptacle, U1 TVS_ESD_USB, U2 AP2112K-3.3, U3 NEO-F10N, U8 CH340C

Commit message: Update datasheet links
Parts:
- L2: value 30Ohm_0603_1.8A -> 30Ohm; symbol SparkFun-Coil:30Ohm_100MHz_0603 -> SparkFun-Coil:30Ohm_0603_1.8A
Changed lines of the file:
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@@
     )
   )
-  (symbol (lib_id "SparkFun-Coil:30Ohm_100MHz_0603") (at 233.68 33.02 0) (unit 1)
+  (symbol (lib_id "SparkFun-Coil:30Ohm_0603_1.8A") (at 233.68 33.02 0) (unit 1)
     (in_bom yes) (on_board yes) (dnp no) (fields_autoplaced)
     (property "Reference" "L2" (at 233.68 24.13 0)
       (effects (font (size 1.27 1.27)))
     )
-    (property "Value" "30Ohm_0603_1.8A" (at 233.68 26.67 0)
+    (property "Value" "30Ohm" (at 233.68 26.67 0)
       (effects (font (size 1.27 1.27)))
     )
@@
       (effects (font (size 1.27 1.27)) hide)
     )
-    (property "Datasheet" "[link text](https://cdn.sparkfun.com/assets/8/a/4/a/5/Kemet_Capacitor_Datasheet.pdf)" (at 88.9 99.06 0)
+    (property "Datasheet" "https://cdn.sparkfun.com/assets/8/a/4/a/5/Kemet_Capacitor_Datasheet.pdf" (at 88.9 99.06 0)
       (effects (font (size 1.27 1.27)) hide)
     )
@@
       (effects (font (size 1.27 1.27)) hide)
     )
-    (property "Datasheet" "[link text](https://cdn.sparkfun.com/assets/8/a/4/a/5/Kemet_Capacitor_Datasheet.pdf)" (at 140.97 99.06 0)
+    (property "Datasheet" "https://cdn.sparkfun.com/assets/8/a/4/a/5/Kemet_Capacitor_Datasheet.pdf" (at 140.97 99.06 0)
       (effects (font (size 1.27 1.27)) hide)
     )
@@
       (effects (font (size 1.27 1.27)) hide)
     )
-    (property "Datasheet" "[link text](https://cdn.sparkfun.com/assets/8/a/4/a/5/Kemet_Capacitor_Datasheet.pdf)" (at 220.98 52.07 0)
+    (property "Datasheet" "https://cdn.sparkfun.com/assets/8/a/4/a/5/Kemet_Capacitor_Datasheet.pdf" (at 220.98 52.07 0)
       (effects (font (size 1.27 1.27)) hide)
     )
@@
       (effects (font (size 1.27 1.27)) hide)
     )
-    (property "Datasheet" "[link text](https://cdn.sparkfun.com/assets/8/a/4/a/5/Kemet_Capacitor_Datasheet.pdf)" (at 100.33 99.06 0)
-      (effects (font (size 1.27 1.27)) hide)
-    )
+    (property "Datasheet" "https://cdn.sparkfun.com/assets/8/a/4/a/5/Kemet_Capacitor_Datasheet.pdf" (at 100.33 99.06 0)
+      (effects (font (size 1.27 1.27)) hide)
+    )
