File: Hardware/SparkFun_NEO-F10N-Connectors.kicad_sch (KiCad schematic)
At the start: 10 parts, among them J2 Conn_01x09, J5 SMA_EdgeMount

Commit message: Update layout and panel files post design review.
Parts:
- added J4: Conn_01x06, SparkFun-Connector:1X06, symbol SparkFun-Connector:Conn_01x06
- added JP8: ~, SparkFun-Jumper:SMT-JUMPER_2_NC_TRACE_SILK, symbol SparkFun-Jumper:SolderJumper_2_Bridged
- C6, C7: symbol SparkFun-Capacitor:47pF_0603_50V_10% -> SparkFun-Capacitor:47pF_0603_50V_5%
Connections:
- net GND: now also J4.6 (Pin_6)
- net RXD: now also J4.3 (Pin_3)
- net TXD: now also J4.2 (Pin_2)
- net +3.3V_A renamed 3.3V
- net 3.3V: now also JP8.2 (B)
- net +5V renamed 5V
- new net: J4.4 (Pin_4), JP8.1 (A)
Other:
- note added: "BlueSMiRF Connector"
- moved on the sheet: R3

Commit message: Update 3D models
Parts:
- C4: Tolerance +80%/-20% -> 20%
- D2, D3: value TVS_ESD_4 -> PESD3V3L4UG
- D6: value TVS_0402 -> PESD0402
- J2: footprint SparkFun-Connector:1X09 -> SparkFun-Connector:1x09
- J4: footprint SparkFun-Connector:1X06 -> SparkFun-Connector:1x06
- J5: value SMA_EdgeMount -> SMA_Edge; footprint SparkFun-Connector:SMA-EDGE -> SparkFun-Connector:SMA_Edge
- JP8: footprint SparkFun-Jumper:SMT-JUMPER_2_NC_TRACE_SILK -> SparkFun-Jumper:Jumper_2_NC_Trace
Connections:
- net GND: no longer J5.1, J5.3, J5.4
- net at C7.1, D6.2 (A2), L1.2: now also J5.1 (In); no longer J5.SIG (In)
